Commit message: lots of misc updates (sry)

File: data/mico.urdf (robot description, URDF)
Before this commit: robot ADA, 16 links, 15 joints
Links:
- link Camera_Collision_Frame: geometry collision mesh filename=package://ada_adjustable_playback/meshes/StructureIO.stl; visual mesh filename=package://ada_adjustable_playback/meshes/structureio.dae
- link mico_link_1: geometry collision mesh filename=package://ada_adjustable_playback/meshes/mico_link_1.dae; visual mesh filename=package://ada_adjustable_playback/meshes/mico_link_1.dae
- link mico_link_2: geometry collision mesh filename=package://ada_adjustable_playback/meshes/mico_link_2.dae; visual mesh filename=package://ada_adjustable_playback/meshes/mico_link_2.dae
- link mico_link_3: geometry collision mesh filename=package://ada_adjustable_playback/meshes/mico_link_3.dae; visual mesh filename=package://ada_adjustable_playback/meshes/mico_link_3.dae
- link mico_link_4: geometry collision mesh filename=package://ada_adjustable_playback/meshes/mico_link_4.dae; visual mesh filename=package://ada_adjustable_playback/meshes/mico_link_4.dae
- link mico_link_5: geometry collision mesh filename=package://ada_adjustable_playback/meshes/mico_link_4.dae; visual mesh filename=package://ada_adjustable_playback/meshes/mico_link_4.dae
- link mico_link_base: geometry collision mesh filename=package://ada_adjustable_playback/meshes/mico_link_base.dae; visual mesh filename=package://ada_adjustable_playback/meshes/mico_link_base.dae
- link mico_link_finger_1: geometry collision mesh filename=package://ada_adjustable_playback/meshes/finger_proximal_li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; visual mesh filename=package://ada_adjustable_playback/meshes/finger_proximal_li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
- link mico_link_finger_2: geometry collision mesh filename=package://ada_adjustable_playback/meshes/finger_proximal_li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; visual mesh filename=package://ada_adjustable_playback/meshes/finger_proximal_li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
- link mico_link_finger_tip_1: geometry collision mesh filename=package://ada_adjustable_playback/meshes/finger_distal_limb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; visual mesh filename=package://ada_adjustable_playback/meshes/finger_distal_limb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
- link mico_link_finger_tip_2: geometry collision mesh filename=package://ada_adjustable_playback/meshes/finger_distal_limb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; visual mesh filename=package://ada_adjustable_playback/meshes/finger_distal_limb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
- link mico_link_hand: geometry collision mesh filename=package://ada_adjustable_playback/meshes/mico_link_hand.dae; visual mesh filename=package://ada_adjustable_playback/meshes/mico_link_hand.dae

Commit message: update more package names

File: data/mico.urdf (robot description, URDF)
Before this commit: robot ADA, 16 links, 15 joints
Links:
- link Camera_Collision_Frame: geometry collision mesh filename=package://harmonic_playback/meshes/StructureIO.stl; visual mesh filename=package://harmonic_playback/meshes/structureio.dae
- link mico_link_1: geometry collision mesh filename=package://harmonic_playback/meshes/mico_link_1.dae; visual mesh filename=package://harmonic_playback/meshes/mico_link_1.dae
- link mico_link_2: geometry collision mesh filename=package://harmonic_playback/meshes/mico_link_2.dae; visual mesh filename=package://harmonic_playback/meshes/mico_link_2.dae
- link mico_link_3: geometry collision mesh filename=package://harmonic_playback/meshes/mico_link_3.dae; visual mesh filename=package://harmonic_playback/meshes/mico_link_3.dae
- link mico_link_4: geometry collision mesh filename=package://harmonic_playback/meshes/mico_link_4.dae; visual mesh filename=package://harmonic_playback/meshes/mico_link_4.dae
- link mico_link_5: geometry collision mesh filename=package://harmonic_playback/meshes/mico_link_4.dae; visual mesh filename=package://harmonic_playback/meshes/mico_link_4.dae
- link mico_link_base: geometry collision mesh filename=package://harmonic_playback/meshes/mico_link_base.dae; visual mesh filename=package://harmonic_playback/meshes/mico_link_base.dae
- link mico_link_finger_1: geometry collision mesh filename=package://harmonic_playback/meshes/finger_proximal_limb_1.d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; visual mesh filename=package://harmonic_playback/meshes/finger_proximal_limb_1.d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
- link mico_link_finger_2: geometry collision mesh filename=package://harmonic_playback/meshes/finger_proximal_limb_1.d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; visual mesh filename=package://harmonic_playback/meshes/finger_proximal_limb_1.d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
- link mico_link_finger_tip_1: geometry collision mesh filename=package://harmonic_playback/meshes/finger_distal_limb_1.dae; visual mesh filename=package://harmonic_playback/meshes/finger_distal_limb_1.dae
- link mico_link_finger_tip_2: geometry collision mesh filename=package://harmonic_playback/meshes/finger_distal_limb_1.dae; visual mesh filename=package://harmonic_playback/meshes/finger_distal_limb_1.dae
- link mico_link_hand: geometry collision mesh filename=package://harmonic_playback/meshes/mico_link_hand.dae; visual mesh filename=package://harmonic_playback/meshes/mico_link_hand.dae

Commit message: add fork tip to mico urdf

File: data/mico.urdf (robot description, URDF)
Before this commit: robot ADA, 16 links, 15 joints
Links:
- added link mico_fork_tip
Joints:
- added joint mico_end_effector_to_fork_tip: type fixed, parent mico_end_effector, child mico_fork_tip, origin xyz=-0.2765016 -0.02133217 -0.0012 rpy=-0.09817476977 1.57079632679 0

Commit message: fix a bunch of dumb bugs

File: data/mico.urdf (robot description, URDF)
Before this commit: robot ADA, 17 links, 16 joints
Links:
- removed link mico_fork_tip
- removed link world
Joints:
- removed joint mico_end_effector_to_fork_tip
- removed joint world_2_base_fixed
